File: Sparkfun Advanced SMD Tutorial/Sparkfun Advanced SMD Tutorial.sch (KiCad schematic (older format))
At the start: 15 parts, among them J1 USB_B_Mini, J2 Conn_01x07, U1 FT230XS

Commit message: Time to assign fottprints to schematic symbols.
Connections:
- net labels added: GNDPWR
- net labels removed: 3V3, 5V
- wire segments 43 -> 45
- no-connect marks 1 -> 3
Changed lines of the file:
@@
 EESchema Schematic File Version 4
+LIBS:Sparkfun Advanced SMD Tutorial-cache
 EELAYER 26 0
 EELAYER END
@@
 	7750 3650 7750 3750
 Text Label 7850 3450 2    50   ~ 0
-3V3
++3V3
 Text Label 7850 3550 2    50   ~ 0
-5V
++5V
 Connection ~ 5150 2650
 Wire Wire Line
@@
 Connection ~ 2400 3650
 NoConn ~ 2700 3450
+NoConn ~ 6650 3750
+NoConn ~ 6650 3850
+$Comp
+L power:PWR_FLAG #FLG0101
+U 1 1 5B426808
+P -450 2550
+F 0 "#FLG0101" H -450 2625 50  0001 C CNN
+F 1 "PWR_FLAG" H -450 2724 50  0000 C CNN
+F 2 "" H -450 2550 50  0001 C CNN
+F 3 "~" H -450 2550 50  0001 C CNN
+	1    -450 2550
+	-1   0    0    1
+$EndComp
+$Comp
+L power:GNDPWR #PWR0111
+U 1 1 5B42689C
+P -50 2550
+F 0 "#PWR0111" H -50 2350 50  0001 C CNN
+F 1 "GNDPWR" H -46 2396 50  0000 C CNN
+F 2 "" H -50 2500 50  0001 C CNN
+F 3 "" H -50 2500 50  0001 C CNN
+	1    -50  2550
+	1    0    0    -1
+$EndComp
+$Comp
+L power:+5V #PWR0112
+U 1 1 5B4269BC
+P -450 2250
+F 0 "#PWR0112" H -450 2100 50  0001 C CNN
+F 1 "+5V" H -435 2423 50  0000 C CNN
+F 2 "" H -450 2250 50  0001 C CNN
+F 3 "" H -450 2250 50  0001 C CNN
+	1    -450 2250
+	1    0    0    -1
+$EndComp
+$Comp
+L power:GND #PWR0114
+U 1 1 5B42727C
+P -50 2250
+F 0 "#PWR0114" H -50 2000 50  0001 C CNN
+F 1 "GND" H -45 2077 50  0000 C CNN
+F 2 "" H -50 2250 50  0001 C CNN
+F 3 "" H -50 2250 50  0001 C CNN
+	1    -50  2250
+	-1   0    0    1
+$EndComp
+Wire Wire Line
+	-50  2250 -50  2550
+Wire Wire Line
+	-450 2550 -450 2250
 $EndSCHEMATC

Commit message: tryin to create my own footprints...
Parts:
- C1, C3: footprint (none) -> Capacitors_SMD:C_0603
- C2: footprint (none) -> Capacitors_SMD:C_1206
- D1, D2: footprint (none) -> LEDs:LED_0603
- J1: footprint (none) -> Connectors:USB_Mini-B
Changed lines of the file:
@@
 F 0 "J1" H 2455 3717 50  0000 C CNN
 F 1 "USB_B_Mini" H 2455 3626 50  0000 C CNN
-F 2 "" H 2550 3200 50  0001 C CNN
+F 2 "Connectors:USB_Mini-B" H 2550 3200 50  0001 C CNN
 F 3 "~" H 2550 3200 50  0001 C CNN
 	1    2400 3250
@@
 F 0 "D1" H 6891 4316 50  0000 C CNN
 F 1 "LED" H 6891 4225 50  0000 C CNN
-F 2 "" H 6900 4100 50  0001 C CNN
+F 2 "LEDs:LED_0603" H 6900 4100 50  0001 C CNN
 F 3 "~" H 6900 4100 50  0001 C CNN
 	1    6900 4100
@@
 F 0 "D2" H 7191 4316 50  0000 C CNN
 F 1 "LED" H 7191 4225 50  0000 C CNN
-F 2 "" H 7200 4100 50  0001 C CNN
+F 2 "LEDs:LED_0603" H 7200 4100 50  0001 C CNN
 F 3 "~" H 7200 4100 50  0001 C CNN
 	1    7200 4100
@@
 F 0 "C1" H 3815 3946 50  0000 L CNN
 F 1 "0.1uF" H 3815 3855 50  0000 L CNN
-F 2 "" H 3738 3750 50  0001 C CNN
+F 2 "Capacitors_SMD:C_0603" H 3738 3750 50  0001 C CNN
 F 3 "~" H 3700 3900 50  0001 C CNN
 	1    3700 3900
@@
 F 0 "C3" H 4765 3946 50  0000 L CNN
 F 1 "0.1uF" H 4765 3855 50  0000 L CNN
-F 2 "" H 4688 3750 50  0001 C CNN
+F 2 "Capacitors_SMD:C_0603" H 4688 3750 50  0001 C CNN
 F 3 "~" H 4650 3900 50  0001 C CNN
 	1    4650 3900
@@
 F 0 "C2" H 4318 3946 50  0000 L CNN
 F 1 "10uF" H 4318 3855 50  0000 L CNN
-F 2 "" H 4238 3750 50  0001 C CNN
+F 2 "Capacitors_SMD:C_1206" H 4238 3750 50  0001 C CNN
 F 3 "~" H 4200 3900 50  0001 C CNN
 	1    4200 3900
