File: Raspberry Pi Expansion Board TEST/Raspberry Pi Expansion Board TEST.kicad_pcb (KiCad board)
At the start: 2 copper layers, 65 x 56 mm, 5 parts, among them P1 Conn_02x20_Odd_Even

Commit message: experimented with creating a board from start to finish (L7805 proj.)
Routing:
- added copper zone on B.Cu, net GND
- added copper zone on F.Cu, net GND
Other:
- outline, holes or cut-outs redrawn
Changed lines of the file:
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@@
-(kicad_pcb (version 20171130) (host pcbnew no-vcs-found-c6d0075~61~ubuntu16.04.1)
+(kicad_pcb (version 20171130) (host pcbnew "(5.0.0-rc3-dev-2-g101b68b61)")
   (general
     (thickness 1.6)
-    (drawings 39)
+    (drawings 32)
     (tracks 0)
     (zones 0)
@@
     (0 F.Cu signal)
     (31 B.Cu signal)
-    (32 B.Adhes user)
     (33 F.Adhes user)
-    (34 B.Paste user)
-    (35 F.Paste user)
-    (36 B.SilkS user)
     (37 F.SilkS user)
-    (38 B.Mask user)
     (39 F.Mask user)
     (40 Dwgs.User user)
@@
     (43 Eco2.User user)
     (44 Edge.Cuts user)
+    (45 Margin user)
+    (46 B.CrtYd user)
+    (47 F.CrtYd user)
+    (49 F.Fab user)
   )
   (setup
@@
     (mod_text_size 1 1)
     (mod_text_width 0.15)
-    (pad_size 2.5 2.5)
-    (pad_drill 2.5)
+    (pad_size 2.7 2.7)
+    (pad_drill 2.7)
     (pad_to_mask_clearance 0)
     (aux_axis_origin 200 150)
@@
       (hpglpennumber 1)
       (hpglpenspeed 20)
-      (hpglpendiameter 15)
+      (hpglpendiameter 15.000000)
       (psnegative false)
       (psa4output false)
@@
       (effects (font (size 1 1) (thickness 0.15)))
     )
-    (pad 1 np_thru_hole circle (at 0 0) (size 2.7 2.7) (drill 2.7) (layers *.Cu *.Mask))
+    (pad "" np_thru_hole circle (at 0 0) (size 2.7 2.7) (drill 2.7) (layers *.Cu *.Mask)
+      (clearance 1.6))
   )
   (module MountingHole:MountingHole_2.7mm_M2.5 (layer F.Cu)
@@
     (fp_circle (center 0 0) (end 2.7 0) (layer Cmts.User) (width 0.15))
     (fp_circle (center 0 0) (end 2.95 0) (layer F.CrtYd) (width 0.05))
-    (pad 1 np_thru_hole circle (at 0 0) (size 2.7 2.7) (drill 2.7) (layers *.Cu *.Mask))
+    (pad "" np_thru_hole circle (at 0 0) (size 2.7 2.7) (drill 2.7) (layers *.Cu *.Mask)
+      (clearance 1.6))
   )
   (module MountingHole:MountingHole_2.7mm_M2.5 (layer F.Cu)
@@
       (effects (font (size 1 1) (thickness 0.15)))
     )
-    (pad 1 np_thru_hole circle (at 0 0 180) (size 2.7 2.7) (drill 2.7) (layers *.Cu *.Mask))
+    (pad "" np_thru_hole circle (at 0 0 180) (size 2.7 2.7) (drill 2.7) (layers *.Cu *.Mask)
+      (clearance 1.6))
   )
   (module MountingHole:MountingHole_2.7mm_M2.5 (layer F.Cu)
@@
     (fp_circle (center 0 0) (end 2.7 0) (layer Cmts.User) (width 0.15))
     (fp_circle (center 0 0) (end 2.95 0) (layer F.CrtYd) (width 0.05))
-    (pad 1 np_thru_hole circle (at 0 0 180) (size 2.7 2.7) (drill 2.7) (layers *.Cu *.Mask))
+    (pad "" np_thru_hole circle (at 0 0 180) (size 2.7 2.7) (drill 2.7) (layers *.Cu *.Mask)
+      (clearance 1.6))
   )
   (gr_line (start 244 146) (end 244 131) (layer Edge.Cuts) (width 0.1))
@@
   (gr_arc (start 245 131) (end 244 131) (angle 180) (layer Edge.Cuts) (width 0.1))
   (gr_arc (start 245 146) (end 246 146) (angle 180) (layer Edge.Cuts) (width 0.1))
-  (gr_arc (start 200.5 131) (end 200 131) (angle 89.9) (layer Edge.Cuts) (width 0.1))
-  (gr_arc (start 204.5 130) (end 205 130) (angle 90) (layer Edge.Cuts) (width 0.1))
-  (gr_arc (start 200.5 113) (end 200.5 113.5) (angle 90) (layer Edge.Cuts) (width 0.1))
-  (gr_arc (start 204.5 114) (end 204.5 113.5) (angle 90) (layer Edge.Cuts) (width 0.1))
   (gr_line (start 200 113) (end 200 131) (layer Dwgs.User) (width 0.1))
-  (gr_line (start 200 97) (end 200 113) (layer Edge.Cuts) (width 0.1))
+  (gr_line (start 200 97) (end 200 130.95) (layer Edge.Cuts) (width 0.1))
   (gr_text DISPLAY (at 202.5 122 90) (layer Dwgs.User)
     (effects (font (size 1 1) (thickness 0.15)))
@@
   (gr_line (start 287 127.55) (end 269.9 127.55) (layer Dwgs.User) (width 0.1))
   (gr_line (start 287 114.45) (end 287 127.55) (layer Dwgs.User) (width 0.1))
-  (gr_line (start 204.5 130.5) (end 200.5 130.5) (layer Edge.Cuts) (width 0.1))
-  (gr_line (start 205 114) (end 205 130) (layer Edge.Cuts) (width 0.1))
-  (gr_line (start 200.5 113.5) (end 204.5 113.5) (layer Edge.Cuts) (width 0.1))
   (gr_line (start 266 147.675) (end 266 131.825) (layer Dwgs.User) (width 0.1))
   (gr_line (start 287 147.675) (end 266 147.675) (layer Dwgs.User) (width 0.1))
@@
     (effects (font (size 2 1.7) (thickness 0.12)) (justify left))
   )
+  (zone (net 3) (net_name GND) (layer F.Cu) (hatch edge 0.508)
+    (connect_pads (clearance 0.508))
+    (min_thickness 0.254)
+    (fill yes (arc_segments 16) (thermal_gap 0.508) (thermal_bridge_width 0.508))
+    (polygon
+      (pts
+        (xy 190.475 85.865) (xy 293.98 87.77) (xy 297.79 182.385) (xy 186.03 178.575)
+      )
+    )
+  )
+  (zone (net 3) (net_name GND) (layer B.Cu) (hatch edge 0.508)
+    (connect_pads (clearance 0.508))
+    (min_thickness 0.254)
+    (fill yes (arc_segments 16) (thermal_gap 0.508) (thermal_bridge_width 0.508))
+    (polygon
+      (pts
+        (xy 182.22 80.785) (xy 304.775 83.325) (xy 315.57 190.64) (xy 176.505 183.02) (xy 177.14 182.385)
+        (xy 175.87 173.495)
+      )
+    )
+  )
 )
