File: componentsearchengine/componentsearchengine.sch (KiCad schematic (older format))
At the start: 1 part, among them Y1 X1G004481001512

Commit message: backup
Parts:
- removed Y1: X1G004481001512, SG7050, symbol X1G004481001512:X1G004481001512
- added X1: X1G0044810050_SG7050CAN_2.048_MHZ, prj_lib_fp:SG0705, symbol project_symbols:X1G0044810050_SG7050CAN_2.048_MHZ
Connections:
- wire segments 8 -> 6
Changed lines of the file:
@@
 EESchema Schematic File Version 4
+LIBS:componentsearchengine-cache
 EELAYER 26 0
 EELAYER END
@@
 $EndDescr
 $Comp
-L X1G004481001512:X1G004481001512 Y1
-U 1 1 5B44EDF9
-P 2350 2550
-F 0 "Y1" H 3000 2815 50  0000 C CNN
-F 1 "X1G004481001512" H 3000 2724 50  0000 C CNN
-F 2 "SG7050" H 3500 2650 50  0001 L CNN
-F 3 "http://uk.rs-online.com/web/p/products/9047821" H 3500 2550 50  0001 L CNN
-F 4 "X1G004481001512, Crystal Oscillator, 40 MHz CMOS 15pF, 4-Pin, 7 x 5 x 1.3mm" H 3500 2450 50  0001 L CNN "Description"
-F 5 "" H 3500 2350 50  0001 L CNN "Height"
-F 6 "Epson Timing" H 3500 2250 50  0001 L CNN "Manufacturer_Name"
-F 7 "X1G004481001512" H 3500 2150 50  0001 L CNN "Manufacturer_Part_Number"
-F 8 "9047821" H 3500 2050 50  0001 L CNN "RS Part Number"
-F 9 "http://uk.rs-online.com/web/p/products/9047821" H 3500 1950 50  0001 L CNN "RS Price/Stock"
-F 10 "X1G004481001512" H 3500 1850 50  0001 L CNN "Arrow Part Number"
-F 11 "http://uk.rs-online.com/web/p/products/9047821" H 3500 1750 50  0001 L CNN "Arrow Price/Stock"
-	1    2350 2550
+L power:+3V3 #PWR0101
+U 1 1 5B44F912
+P 2300 2100
+F 0 "#PWR0101" H 2300 1950 50  0001 C CNN
+F 1 "+3V3" H 2315 2273 50  0000 C CNN
+F 2 "" H 2300 2100 50  0001 C CNN
+F 3 "" H 2300 2100 50  0001 C CNN
+	1    2300 2100
 	1    0    0    -1
 $EndComp
 $Comp
-L power:+3V3 #PWR0101
-U 1 1 5B44F912
-P 2350 2150
-F 0 "#PWR0101" H 2350 2000 50  0001 C CNN
-F 1 "+3V3" H 2365 2323 50  0000 C CNN
-F 2 "" H 2350 2150 50  0001 C CNN
-F 3 "" H 2350 2150 50  0001 C CNN
-	1    2350 2150
+L power:GND #PWR0102
+U 1 1 5B44F95D
+P 3750 2650
+F 0 "#PWR0102" H 3750 2400 50  0001 C CNN
+F 1 "GND" H 3755 2477 50  0000 C CNN
+F 2 "" H 3750 2650 50  0001 C CNN
+F 3 "" H 3750 2650 50  0001 C CNN
+	1    3750 2650
+	1    0    0    -1
+$EndComp
+$Comp
+L power:PWR_FLAG #FLG01
+U 1 1 5B451778
+P -150 2150
+F 0 "#FLG01" H -150 2225 50  0001 C CNN
+F 1 "PWR_FLAG" V -150 2278 50  0000 L CNN
+F 2 "" H -150 2150 50  0001 C CNN
+F 3 "~" H -150 2150 50  0001 C CNN
+	1    -150 2150
+	0    -1   -1   0
+$EndComp
+$Comp
+L power:+3V3 #PWR01
+U 1 1 5B451783
+P -150 2150
+F 0 "#PWR01" H -150 2000 50  0001 C CNN
+F 1 "+3V3" H -135 2323 50  0000 C CNN
+F 2 "" H -150 2150 50  0001 C CNN
+F 3 "" H -150 2150 50  0001 C CNN
+	1    -150 2150
+	1    0    0    -1
+$EndComp
+$Comp
+L power:PWR_FLAG #FLG02
+U 1 1 5B45178E
+P -150 2450
+F 0 "#FLG02" H -150 2525 50  0001 C CNN
+F 1 "PWR_FLAG" V -150 2578 50  0000 L CNN
+F 2 "" H -150 2450 50  0001 C CNN
+F 3 "~" H -150 2450 50  0001 C CNN
+	1    -150 2450
+	0    -1   -1   0
+$EndComp
+$Comp
+L power:GND #PWR02
+U 1 1 5B451799
+P -150 2450
+F 0 "#PWR02" H -150 2200 50  0001 C CNN
+F 1 "GND" H -145 2277 50  0000 C CNN
+F 2 "" H -150 2450 50  0001 C CNN
+F 3 "" H -150 2450 50  0001 C CNN
+	1    -150 2450
 	1    0    0    -1
 $EndComp
 Wire Wire Line
-	2350 2150 2350 2450
+	2300 2100 2300 2400
 Wire Wire Line
-	2350 2150 3800 2150
+	2300 2400 2550 2400
 Wire Wire Line
-	3800 2150 3800 2650
+	3750 2650 3750 2550
 Wire Wire Line
-	3800 2650 3650 2650
-Connection ~ 2350 2150
+	3750 2550 3650 2550
 Wire Wire Line
-	2350 2650 2350 2750
+	3650 2400 3950 2400
+NoConn ~ 3950 2400
 $Comp
-L power:GND #PWR0102
-U 1 1 5B44F95D
-P 2350 2900
-F 0 "#PWR0102" H 2350 2650 50  0001 C CNN
-F 1 "GND" H 2355 2727 50  0000 C CNN
-F 2 "" H 2350 2900 50  0001 C CNN
-F 3 "" H 2350 2900 50  0001 C CNN
-	1    2350 2900
+L project_symbols:X1G0044810050_SG7050CAN_2.048_MHZ X1
+U 1 1 5B4519FE
+P 3100 2500
+F 0 "X1" H 3100 2825 50  0000 C CNN
+F 1 "X1G0044810050_SG7050CAN_2.048_MHZ" H 3100 2734 50  0000 C CNN
+F 2 "prj_lib_fp:SG0705" H 3050 2500 50  0001 C CNN
+F 3 "http://www.farnell.com/datasheets/1841779.pdf" H 2400 2950 50  0001 C CNN
+F 4 "2442953" H 1600 3050 50  0001 C CNN "Farnell Part"
+F 5 "http://se.farnell.com/epson/x1g0044810050-sg7050can-2-048-mhz/oscillator-spxo-sg7050can-2-048/dp/2442953" H 3800 3150 50  0001 C CNN "Farnell URL"
+	1    3100 2500
 	1    0    0    -1
 $EndComp
-$Comp
-L power:PWR_FLAG #FLG0101
-U 1 1 5B44FA02
-P 2350 2450
-F 0 "#FLG0101" H 2350 2525 50  0001 C CNN
-F 1 "PWR_FLAG" V 2350 2578 50  0000 L CNN
-F 2 "" H 2350 2450 50  0001 C CNN
-F 3 "~" H 2350 2450 50  0001 C CNN
-	1    2350 2450
-	0    -1   -1   0
-$EndComp
-Connection ~ 2350 2450
 Wire Wire Line
-	2350 2450 2350 2550
-$Comp
-L power:PWR_FLAG #FLG0102
-U 1 1 5B44FA1B
-P 2350 2750
-F 0 "#FLG0102" H 2350 2825 50  0001 C CNN
-F 1 "PWR_FLAG" V 2350 2878 50  0000 L CNN
-F 2 "" H 2350 2750 50  0001 C CNN
-F 3 "~" H 2350 2750 50  0001 C CNN
-	1    2350 2750
-	0    -1   -1   0
-$EndComp
-Connection ~ 2350 2750
-Wire Wire Line
-	2350 2750 2350 2900
-Wire Wire Line
-	3650 2550 3900 2550
-NoConn ~ 3900 2550
+	2550 2550 2550 2400
+Connection ~ 2550 2400
 $EndSCHEMATC

Commit message: plz no crash now.
Parts:
- added J1: Conn_02x03_Counter_Clockwise, Pin_Headers:Pin_Header_Straight_2x03_Pitch2.54mm, symbol Connector_Generic:Conn_02x03_Counter_Clockwise
- added U1: ADS1299-4PAG, prj_lib_fp:xQFP_64_to_2.54mm_adapter, symbol ADS1299-4PAG:ADS1299-4PAG
Changed lines of the file:
@@
 F 1 "PWR_FLAG" V -150 2278 50  0000 L CNN
 F 2 "" H -150 2150 50  0001 C CNN
-F 3 "~" H -150 2150 50  0001 C CNN
+F 3 "" H -150 2150 50  0001 C CNN
 	1    -150 2150
 	0    -1   -1   0
@@
 F 1 "PWR_FLAG" V -150 2578 50  0000 L CNN
 F 2 "" H -150 2450 50  0001 C CNN
-F 3 "~" H -150 2450 50  0001 C CNN
+F 3 "" H -150 2450 50  0001 C CNN
 	1    -150 2450
 	0    -1   -1   0
@@
 	2550 2550 2550 2400
 Connection ~ 2550 2400
+$Comp
+L ADS1299-4PAG:ADS1299-4PAG U1
+U 1 1 5B454C4D
+P 2550 4800
+F 0 "U1" H 2550 6567 50  0000 C CNN
+F 1 "ADS1299-4PAG" H 2550 6476 50  0000 C CNN
+F 2 "prj_lib_fp:xQFP_64_to_2.54mm_adapter" H 4050 5900 50  0001 L BNN
+F 3 "http://www.ti.com/lit/ds/symlink/ads1299-4.pdf" H 4000 6200 50  0001 L BNN
+F 4 "Low-Noise, 4-Channel, 24-Bit Analog-to-Digital Converter for Biopotential Measurements 64-TQFP -40 to 85" H 4000 6100 50  0001 L BNN "Description"
+F 5 "2707750" H 1947 6605 50  0001 L BNN "Farnell Part"
+F 6 "http://se.farnell.com/texas-instruments/ads1299-4pag/adc-quad-24-bits-16ksps-tqfp-64/dp/2707750" H 1847 6505 50  0001 L BNN "Farnell URL"
+	1    2550 4800
+	1    0    0    -1
+$EndComp
+$Comp
+L Connector_Generic:Conn_02x03_Counter_Clockwise J1
+U 1 1 5B4550CF
+P 4450 4450
+F 0 "J1" H 4500 4767 50  0000 C CNN
+F 1 "Conn_02x03_Counter_Clockwise" H 4500 4676 50  0000 C CNN
+F 2 "Pin_Headers:Pin_Header_Straight_2x03_Pitch2.54mm" H 4450 4450 50  0001 C CNN
+F 3 "~" H 4450 4450 50  0001 C CNN
+	1    4450 4450
+	1    0    0    -1
+$EndComp
 $EndSCHEMATC

Commit message: Goodnight.
Connections:
- no-connect marks 1 -> 0
Changed lines of the file:
@@
 L power:+3V3 #PWR0101
 U 1 1 5B44F912
-P 2300 2100
-F 0 "#PWR0101" H 2300 1950 50  0001 C CNN
-F 1 "+3V3" H 2315 2273 50  0000 C CNN
-F 2 "" H 2300 2100 50  0001 C CNN
-F 3 "" H 2300 2100 50  0001 C CNN
-	1    2300 2100
+P 2950 3350
+F 0 "#PWR0101" H 2950 3200 50  0001 C CNN
+F 1 "+3V3" H 2965 3523 50  0000 C CNN
+F 2 "" H 2950 3350 50  0001 C CNN
+F 3 "" H 2950 3350 50  0001 C CNN
+	1    2950 3350
 	1    0    0    -1
 $EndComp
@@
 L power:GND #PWR0102
 U 1 1 5B44F95D
-P 3750 2650
-F 0 "#PWR0102" H 3750 2400 50  0001 C CNN
-F 1 "GND" H 3755 2477 50  0000 C CNN
-F 2 "" H 3750 2650 50  0001 C CNN
-F 3 "" H 3750 2650 50  0001 C CNN
-	1    3750 2650
+P 4400 3900
+F 0 "#PWR0102" H 4400 3650 50  0001 C CNN
+F 1 "GND" H 4405 3727 50  0000 C CNN
+F 2 "" H 4400 3900 50  0001 C CNN
+F 3 "" H 4400 3900 50  0001 C CNN
+	1    4400 3900
 	1    0    0    -1
 $EndComp
@@
 $EndComp
 Wire Wire Line
-	2300 2100 2300 2400
+	2950 3350 2950 3650
 Wire Wire Line
-	2300 2400 2550 2400
+	2950 3650 3200 3650
 Wire Wire Line
-	3750 2650 3750 2550
+	4400 3900 4400 3800
 Wire Wire Line
-	3750 2550 3650 2550
-Wire Wire Line
-	3650 2400 3950 2400
-NoConn ~ 3950 2400
+	4400 3800 4300 3800
 $Comp
 L project_symbols:X1G0044810050_SG7050CAN_2.048_MHZ X1
 U 1 1 5B4519FE
-P 3100 2500
-F 0 "X1" H 3100 2825 50  0000 C CNN
-F 1 "X1G0044810050_SG7050CAN_2.048_MHZ" H 3100 2734 50  0000 C CNN
-F 2 "prj_lib_fp:SG0705" H 3050 2500 50  0001 C CNN
-F 3 "http://www.farnell.com/datasheets/1841779.pdf" H 2400 2950 50  0001 C CNN
-F 4 "2442953" H 1600 3050 50  0001 C CNN "Farnell Part"
-F 5 "http://se.farnell.com/epson/x1g0044810050-sg7050can-2-048-mhz/oscillator-spxo-sg7050can-2-048/dp/2442953" H 3800 3150 50  0001 C CNN "Farnell URL"
-	1    3100 2500
+P 3750 3750
+F 0 "X1" H 3750 4075 50  0000 C CNN
+F 1 "X1G0044810050_SG7050CAN_2.048_MHZ" H 3750 3984 50  0000 C CNN
+F 2 "prj_lib_fp:SG0705" H 3700 3750 50  0001 C CNN
+F 3 "http://www.farnell.com/datasheets/1841779.pdf" H 3050 4200 50  0001 C CNN
+F 4 "2442953" H 2250 4300 50  0001 C CNN "Farnell Part"
+F 5 "http://se.farnell.com/epson/x1g0044810050-sg7050can-2-048-mhz/oscillator-spxo-sg7050can-2-048/dp/2442953" H 4450 4400 50  0001 C CNN "Farnell URL"
+	1    3750 3750
 	1    0    0    -1
 $EndComp
 Wire Wire Line
-	2550 2550 2550 2400
-Connection ~ 2550 2400
+	3200 3800 3200 3650
+Connection ~ 3200 3650
 $Comp
 L ADS1299-4PAG:ADS1299-4PAG U1
 U 1 1 5B454C4D
-P 2550 4800
-F 0 "U1" H 2550 6567 50  0000 C CNN
-F 1 "ADS1299-4PAG" H 2550 6476 50  0000 C CNN
-F 2 "prj_lib_fp:xQFP_64_to_2.54mm_adapter" H 4050 5900 50  0001 L BNN
-F 3 "http://www.ti.com/lit/ds/symlink/ads1299-4.pdf" H 4000 6200 50  0001 L BNN
-F 4 "Low-Noise, 4-Channel, 24-Bit Analog-to-Digital Converter for Biopotential Measurements 64-TQFP -40 to 85" H 4000 6100 50  0001 L BNN "Description"
-F 5 "2707750" H 1947 6605 50  0001 L BNN "Farnell Part"
-F 6 "http://se.farnell.com/texas-instruments/ads1299-4pag/adc-quad-24-bits-16ksps-tqfp-64/dp/2707750" H 1847 6505 50  0001 L BNN "Farnell URL"
-	1    2550 4800
+P 6000 3050
+F 0 "U1" H 6000 4817 50  0000 C CNN
+F 1 "ADS1299-4PAG" H 6000 4726 50  0000 C CNN
+F 2 "prj_lib_fp:xQFP_64_to_2.54mm_adapter" H 7500 4150 50  0001 L BNN
+F 3 "http://www.ti.com/lit/ds/symlink/ads1299-4.pdf" H 7450 4450 50  0001 L BNN
+F 4 "Low-Noise, 4-Channel, 24-Bit Analog-to-Digital Converter for Biopotential Measurements 64-TQFP -40 to 85" H 7450 4350 50  0001 L BNN "Description"
+F 5 "2707750" H 5397 4855 50  0001 L BNN "Farnell Part"
+F 6 "http://se.farnell.com/texas-instruments/ads1299-4pag/adc-quad-24-bits-16ksps-tqfp-64/dp/2707750" H 5297 4755 50  0001 L BNN "Farnell URL"
+	1    6000 3050
 	1    0    0    -1
 $EndComp
@@
 	1    0    0    -1
 $EndComp
+Wire Wire Line
+	4300 3650 5100 3650
 $EndSCHEMATC
