File: mobilt_eeg_frontend-exjobb2018/mobilt_eeg_frontend-exjobb2018.sch (KiCad schematic (older format))
At the start: 6 parts, among them P1 Conn_02x20_Odd_Even

Commit message: plz no crash now.
Parts:
- removed U?: CAT24C256, symbol Memory_EEPROM:CAT24C256
- added C1: 0.1uF, Capacitors_SMD:C_0805_HandSoldering, symbol Device:C_Small
- added X1: X1G0044810050_SG7050CAN_2.048_MHZ, prj_lib_fp:SG0705, symbol project_symbols:X1G0044810050_SG7050CAN_2.048_MHZ
Connections:
- wire segments 52 -> 63
- no-connect marks 0 -> 31
Changed lines of the file:
@@
 	2300 2300 2400 2300
 Connection ~ 2300 3000
-Connection ~ 2200 1100
 Wire Wire Line
 	2200 1900 2400 1900
-Wire Wire Line
-	2200 1100 2400 1100
-Wire Wire Line
-	2200 950  2200 1100
-$Comp
-L power:+3.3V #PWR04
-U 1 1 580C1BC1
-P 2200 950
-F 0 "#PWR04" H 2200 800 50  0001 C CNN
-F 1 "+3.3V" H 2200 1090 50  0000 C CNN
-F 2 "" H 2200 950 50  0000 C CNN
-F 3 "" H 2200 950 50  0000 C CNN
-	1    2200 950
-	1    0    0    -1
-$EndComp
 Wire Wire Line
 	2300 1500 2400 1500
@@
 	2300 3000 2300 3150
 Wire Wire Line
-	2200 1100 2200 1900
-Wire Wire Line
 	2300 2300 2300 3000
 Wire Wire Line
 	3000 1700 3000 2000
 $Comp
-L Memory_EEPROM:CAT24C256 U?
-U 1 1 5B4385DA
-P 1550 4050
-F 0 "U?" H 1550 4528 50  0000 C CNN
-F 1 "CAT24C256" H 1550 4437 50  0000 C CNN
-F 2 "" H 1550 4050 50  0001 C CNN
-F 3 "https://www.onsemi.cn/PowerSolutions/document/CAT24C256-D.PDF" H 1550 4050 50  0001 C CNN
-	1    1550 4050
-	1    0    0    -1
-$EndComp
+L project_symbols:X1G0044810050_SG7050CAN_2.048_MHZ X1
+U 1 1 5B452FB5
+P 5650 2500
+F 0 "X1" H 5650 2825 50  0000 C CNN
+F 1 "X1G0044810050_SG7050CAN_2.048_MHZ" H 5650 2734 50  0000 C CNN
+F 2 "prj_lib_fp:SG0705" H 5600 2500 50  0001 C CNN
+F 3 "http://www.farnell.com/datasheets/1841779.pdf" H 4950 2950 50  0001 C CNN
+F 4 "2442953" H 4150 3050 50  0001 C CNN "Farnell Part"
+F 5 "http://se.farnell.com/epson/x1g0044810050-sg7050can-2-048-mhz/oscillator-spxo-sg7050can-2-048/dp/2442953" H 6350 3150 50  0001 C CNN "Farnell URL"
+	1    5650 2500
+	1    0    0    -1
+$EndComp
+$Comp
+L power:+3.3V #PWR0101
+U 1 1 5B45455D
+P -350 950
+F 0 "#PWR0101" H -350 800 50  0001 C CNN
+F 1 "+3.3V" H -350 1090 50  0000 C CNN
+F 2 "" H -350 950 50  0000 C CNN
+F 3 "" H -350 950 50  0000 C CNN
+	1    -350 950
+	1    0    0    -1
+$EndComp
+$Comp
+L power:+5V #PWR0102
+U 1 1 5B454586
+P -800 950
+F 0 "#PWR0102" H -800 800 50  0001 C CNN
+F 1 "+5V" H -800 1090 50  0000 C CNN
+F 2 "" H -800 950 50  0000 C CNN
+F 3 "" H -800 950 50  0000 C CNN
+	1    -800 950
+	1    0    0    -1
+$EndComp
+Wire Wire Line
+	2400 1100 2200 1100
+NoConn ~ 2200 1100
+NoConn ~ 2200 1900
+$Comp
+L power:PWR_FLAG #FLG0101
+U 1 1 5B457AAB
+P -800 1150
+F 0 "#FLG0101" H -800 1225 50  0001 C CNN
+F 1 "PWR_FLAG" H -800 1323 50  0000 C CNN
+F 2 "" H -800 1150 50  0001 C CNN
+F 3 "~" H -800 1150 50  0001 C CNN
+	1    -800 1150
+	-1   0    0    1
+$EndComp
+$Comp
+L power:PWR_FLAG #FLG0102
+U 1 1 5B457AD5
+P -350 1150
+F 0 "#FLG0102" H -350 1225 50  0001 C CNN
+F 1 "PWR_FLAG" H -350 1323 50  0000 C CNN
+F 2 "" H -350 1150 50  0001 C CNN
+F 3 "~" H -350 1150 50  0001 C CNN
+	1    -350 1150
+	-1   0    0    1
+$EndComp
+Wire Wire Line
+	-350 1150 -350 950
+Wire Wire Line
+	-800 950  -800 1150
+$Comp
+L power:+3.3V #PWR0103
+U 1 1 5B45A84F
+P 4750 2200
+F 0 "#PWR0103" H 4750 2050 50  0001 C CNN
+F 1 "+3.3V" H 4750 2340 50  0000 C CNN
+F 2 "" H 4750 2200 50  0000 C CNN
+F 3 "" H 4750 2200 50  0000 C CNN
+	1    4750 2200
+	1    0    0    -1
+$EndComp
+Wire Wire Line
+	4750 2200 4750 2400
+Wire Wire Line
+	4750 2400 5100 2400
+Wire Wire Line
+	5100 2550 5100 2400
+Connection ~ 5100 2400
+$Comp
+L power:GND #PWR0104
+U 1 1 5B45C725
+P 6300 2900
+F 0 "#PWR0104" H 6300 2650 50  0001 C CNN
+F 1 "GND" H 6300 2750 50  0000 C CNN
+F 2 "" H 6300 2900 50  0000 C CNN
+F 3 "" H 6300 2900 50  0000 C CNN
+	1    6300 2900
+	1    0    0    -1
+$EndComp
+Wire Wire Line
+	6300 2550 6200 2550
+Wire Wire Line
+	6200 2400 6500 2400
+NoConn ~ 6500 2400
+NoConn ~ 1250 1200
+NoConn ~ 1250 1300
+NoConn ~ 1250 1400
+NoConn ~ 1250 1600
+NoConn ~ 1250 1700
+NoConn ~ 1250 1800
+NoConn ~ 1250 2000
+NoConn ~ 1250 2100
+NoConn ~ 1250 2200
+NoConn ~ 1250 2400
+NoConn ~ 1250 2500
+NoConn ~ 1250 2600
+NoConn ~ 1250 2700
+NoConn ~ 1250 2800
+NoConn ~ 1250 2900
+NoConn ~ 3950 1400
+NoConn ~ 3950 1500
+NoConn ~ 3950 1600
+NoConn ~ 3950 1800
+NoConn ~ 3950 1900
+NoConn ~ 3950 2100
+NoConn ~ 3950 2200
+NoConn ~ 3950 2300
+NoConn ~ 3950 2400
+NoConn ~ 3950 2600
+NoConn ~ 3950 2800
+NoConn ~ 3950 2900
+NoConn ~ 3950 3000
+$Comp
+L Device:C_Small C1
+U 1 1 5B46310B
+P 5650 2800
+F 0 "C1" V 5750 2800 50  0000 C CNN
+F 1 "0.1uF" V 5550 2800 50  0000 C CNN
+F 2 "Capacitors_SMD:C_0805_HandSoldering" H 5650 2800 50  0001 C CNN
+F 3 "~" H 5650 2800 50  0001 C CNN
+	1    5650 2800
+	0    -1   -1   0
+$EndComp
+Wire Wire Line
+	6300 2550 6300 2800
+Wire Wire Line
+	5750 2800 6300 2800
+Connection ~ 6300 2800
+Wire Wire Line
+	6300 2800 6300 2900
+Wire Wire Line
+	5550 2800 5100 2800
+Wire Wire Line
+	5100 2800 5100 2550
+Connection ~ 5100 2550
+$Comp
+L power:GND #PWR0105
+U 1 1 5B467931
+P -1150 1150
+F 0 "#PWR0105" H -1150 900 50  0001 C CNN
+F 1 "GND" H -1150 1000 50  0000 C CNN
+F 2 "" H -1150 1150 50  0000 C CNN
+F 3 "" H -1150 1150 50  0000 C CNN
+	1    -1150 1150
+	1    0    0    -1
+$EndComp
+$Comp
+L power:PWR_FLAG #FLG0103
+U 1 1 5B467A40
+P -1150 950
+F 0 "#FLG0103" H -1150 1025 50  0001 C CNN
+F 1 "PWR_FLAG" H -1150 1123 50  0000 C CNN
+F 2 "" H -1150 950 50  0001 C CNN
+F 3 "~" H -1150 950 50  0001 C CNN
+	1    -1150 950
+	1    0    0    -1
+$EndComp
+Wire Wire Line
+	-1150 950  -1150 1150
 $EndSCHEMATC

Commit message: Goodnight.
Parts:
- added U1: ADS1299-4PAG, xQFP_64_to_2.54mm_adapter, symbol project_symbols:ADS1299-4PAG
Connections:
- net labels added: +3V3, GPIO1, GPIO2, GPIO3, GPIO4
- wire segments 63 -> 73
- no-connect marks 31 -> 26
Changed lines of the file:
@@
 Connection ~ 2300 3000
 Wire Wire Line
-	2200 1900 2400 1900
+	1950 1900 2400 1900
 Wire Wire Line
 	2300 1500 2400 1500
@@
 L project_symbols:X1G0044810050_SG7050CAN_2.048_MHZ X1
 U 1 1 5B452FB5
-P 5650 2500
-F 0 "X1" H 5650 2825 50  0000 C CNN
-F 1 "X1G0044810050_SG7050CAN_2.048_MHZ" H 5650 2734 50  0000 C CNN
-F 2 "prj_lib_fp:SG0705" H 5600 2500 50  0001 C CNN
-F 3 "http://www.farnell.com/datasheets/1841779.pdf" H 4950 2950 50  0001 C CNN
-F 4 "2442953" H 4150 3050 50  0001 C CNN "Farnell Part"
-F 5 "http://se.farnell.com/epson/x1g0044810050-sg7050can-2-048-mhz/oscillator-spxo-sg7050can-2-048/dp/2442953" H 6350 3150 50  0001 C CNN "Farnell URL"
-	1    5650 2500
+P 6950 6450
+F 0 "X1" H 6950 6775 50  0000 C CNN
+F 1 "X1G0044810050_SG7050CAN_2.048_MHZ" H 6950 6684 50  0000 C CNN
+F 2 "prj_lib_fp:SG0705" H 6900 6450 50  0001 C CNN
+F 3 "http://www.farnell.com/datasheets/1841779.pdf" H 6250 6900 50  0001 C CNN
+F 4 "2442953" H 5450 7000 50  0001 C CNN "Farnell Part"
+F 5 "http://se.farnell.com/epson/x1g0044810050-sg7050can-2-048-mhz/oscillator-spxo-sg7050can-2-048/dp/2442953" H 7650 7100 50  0001 C CNN "Farnell URL"
+	1    6950 6450
 	1    0    0    -1
 $EndComp
@@
 $EndComp
 Wire Wire Line
-	2400 1100 2200 1100
-NoConn ~ 2200 1100
-NoConn ~ 2200 1900
+	2400 1100 1950 1100
+NoConn ~ 1950 1100
+NoConn ~ 1950 1900
 $Comp
 L power:PWR_FLAG #FLG0101
@@
 L power:+3.3V #PWR0103
 U 1 1 5B45A84F
-P 4750 2200
-F 0 "#PWR0103" H 4750 2050 50  0001 C CNN
-F 1 "+3.3V" H 4750 2340 50  0000 C CNN
-F 2 "" H 4750 2200 50  0000 C CNN
-F 3 "" H 4750 2200 50  0000 C CNN
-	1    4750 2200
-	1    0    0    -1
-$EndComp
-Wire Wire Line
-	4750 2200 4750 2400
-Wire Wire Line
-	4750 2400 5100 2400
-Wire Wire Line
-	5100 2550 5100 2400
-Connection ~ 5100 2400
+P 6050 6150
+F 0 "#PWR0103" H 6050 6000 50  0001 C CNN
+F 1 "+3.3V" H 6050 6290 50  0000 C CNN
+F 2 "" H 6050 6150 50  0000 C CNN
+F 3 "" H 6050 6150 50  0000 C CNN
+	1    6050 6150
+	1    0    0    -1
+$EndComp
+Wire Wire Line
+	6050 6150 6050 6350
+Wire Wire Line
+	6050 6350 6400 6350
+Wire Wire Line
+	6400 6500 6400 6350
+Connection ~ 6400 6350
 $Comp
 L power:GND #PWR0104
 U 1 1 5B45C725
-P 6300 2900
-F 0 "#PWR0104" H 6300 2650 50  0001 C CNN
-F 1 "GND" H 6300 2750 50  0000 C CNN
-F 2 "" H 6300 2900 50  0000 C CNN
-F 3 "" H 6300 2900 50  0000 C CNN
-	1    6300 2900
-	1    0    0    -1
-$EndComp
-Wire Wire Line
-	6300 2550 6200 2550
-Wire Wire Line
-	6200 2400 6500 2400
-NoConn ~ 6500 2400
+P 7600 6850
+F 0 "#PWR0104" H 7600 6600 50  0001 C CNN
+F 1 "GND" H 7600 6700 50  0000 C CNN
+F 2 "" H 7600 6850 50  0000 C CNN
+F 3 "" H 7600 6850 50  0000 C CNN
+	1    7600 6850
+	1    0    0    -1
+$EndComp
+Wire Wire Line
+	7600 6500 7500 6500
 NoConn ~ 1250 1200
 NoConn ~ 1250 1300
@@
 NoConn ~ 1250 1700
 NoConn ~ 1250 1800
-NoConn ~ 1250 2000
-NoConn ~ 1250 2100
-NoConn ~ 1250 2200
 NoConn ~ 1250 2400
 NoConn ~ 1250 2500
@@
 NoConn ~ 3950 1900
 NoConn ~ 3950 2100
-NoConn ~ 3950 2200
 NoConn ~ 3950 2300
 NoConn ~ 3950 2400
@@
 L Device:C_Small C1
 U 1 1 5B46310B
-P 5650 2800
-F 0 "C1" V 5750 2800 50  0000 C CNN
-F 1 "0.1uF" V 5550 2800 50  0000 C CNN
-F 2 "Capacitors_SMD:C_0805_HandSoldering" H 5650 2800 50  0001 C CNN
-F 3 "~" H 5650 2800 50  0001 C CNN
-	1    5650 2800
+P 6950 6750
+F 0 "C1" V 7050 6750 50  0000 C CNN
+F 1 "0.1uF" V 6850 6750 50  0000 C CNN
+F 2 "Capacitors_SMD:C_0805_HandSoldering" H 6950 6750 50  0001 C CNN
+F 3 "~" H 6950 6750 50  0001 C CNN
+	1    6950 6750
 	0    -1   -1   0
 $EndComp
 Wire Wire Line
-	6300 2550 6300 2800
-Wire Wire Line
-	5750 2800 6300 2800
-Connection ~ 6300 2800
-Wire Wire Line
-	6300 2800 6300 2900
-Wire Wire Line
-	5550 2800 5100 2800
-Wire Wire Line
-	5100 2800 5100 2550
-Connection ~ 5100 2550
+	7600 6500 7600 6750
+Wire Wire Line
+	7050 6750 7600 6750
+Connection ~ 7600 6750
+Wire Wire Line
+	7600 6750 7600 6850
+Wire Wire Line
+	6850 6750 6400 6750
+Wire Wire Line
+	6400 6750 6400 6500
+Connection ~ 6400 6500
 $Comp
 L power:GND #PWR0105
@@
 Wire Wire Line
 	-1150 950  -1150 1150
+Wire Wire Line
+	7500 6350 9200 6350
+$Comp
+L project_symbols:ADS1299-4PAG U1
+U 1 1 5B462F68
+P 10100 5750
+F 0 "U1" H 10100 7517 50  0000 C CNN
+F 1 "ADS1299-4PAG" H 10100 7426 50  0000 C CNN
+F 2 "xQFP_64_to_2.54mm_adapter" H 11600 6850 50  0001 L BNN
+F 3 "http://www.ti.com/lit/ds/symlink/ads1299-4.pdf" H 11550 7150 50  0001 L BNN
+F 4 "Low-Noise, 4-Channel, 24-Bit Analog-to-Digital Converter for Biopotential Measurements 64-TQFP -40 to 85" H 11550 7050 50  0001 L BNN "Description"
+F 5 "2707750" H 9497 7555 50  0001 L BNN "Farnell Part"
+F 6 "http://se.farnell.com/texas-instruments/ads1299-4pag/adc-quad-24-bits-16ksps-tqfp-64/dp/2707750" H 9397 7455 50  0001 L BNN "Farnell URL"
+	1    10100 5750
+	1    0    0    -1
+$EndComp
+Text Label 8350 6050 0    50   ~ 0
+GPIO10(SPI0_MOSI)
+Wire Wire Line
+	8350 6050 9200 6050
+Text Label 11750 5150 2    50   ~ 0
+GPIO9(SPI0_MISO)
+Wire Wire Line
+	11000 5150 11750 5150
+Wire Wire Line
+	9200 6650 8350 6650
+Text Label 8350 6650 0    50   ~ 0
+GPIO11(SPI0_SCK)
+Text Label 8350 6550 0    50   ~ 0
+GPIO8(SPI0_CE_N)
+Wire Wire Line
+	8350 6550 9200 6550
+Text Label 11750 4850 2    50   ~ 0
+GPIO4
+Text Label 11750 4950 2    50   ~ 0
+GPIO3
+Text Label 11750 5050 2    50   ~ 0
+GPIO2
+Text Label 11750 5250 2    50   ~ 0
+GPIO1
+Wire Wire Line
+	11000 5250 11750 5250
+Wire Wire Line
+	11750 4950 11000 4950
+Wire Wire Line
+	11000 4850 11750 4850
+Wire Wire Line
+	11000 5050 11750 5050
+Text Label 1950 1100 0    50   ~ 0
++3V3
+Text Label 1950 1900 0    50   ~ 0
++3V3
+$Comp
+L power:GND #PWR0106
+U 1 1 5B479C6F
+P 12150 4500
+F 0 "#PWR0106" H 12150 4250 50  0001 C CNN
+F 1 "GND" H 12150 4350 50  0000 C CNN
+F 2 "" H 12150 4500 50  0000 C CNN
+F 3 "" H 12150 4500 50  0000 C CNN
+	1    12150 4500
+	1    0    0    -1
+$EndComp
+$Comp
+L power:GND #PWR?
+U 1 1 5B47B937
+P 11100 7150
+F 0 "#PWR?" H 11100 6900 50  0001 C CNN
+F 1 "GND" H 11100 7000 50  0000 C CNN
+F 2 "" H 11100 7150 50  0000 C CNN
+F 3 "" H 11100 7150 50  0000 C CNN
+	1    11100 7150
+	1    0    0    -1
+$EndComp
+Wire Wire Line
+	11000 7050 11100 7050
+Wire Wire Line
+	11100 7050 11100 7150
 $EndSCHEMATC

Commit message: did another bloody tutorial...
Parts:
- added J1: Conn_02x04_Odd_Even, Pin_Headers:Pin_Header_Straight_2x04_Pitch2.54mm, symbol Connector_Generic:Conn_02x04_Odd_Even
- added R1, R2: 10k, Resistors_SMD:R_0805_HandSoldering, symbol Device:R
- U1: footprint xQFP_64_to_2.54mm_adapter -> prj_lib_fp:xQFP_64_to_2.54mm_adapter
Connections:
- net labels added: DVDD, GNDD, IN1_N, IN1_P, ~PWDN, ~RESET
- net labels removed: GND
- wire segments 73 -> 92
- no-connect marks 26 -> 64
Other:
- note added: "ADC GPIO Header\n"
- note added: "External Oscillator"
- note added: "RESET can be trig'd via SPI cmd.\nPWDN only possible in HW."

Commit message: added electrode intermediate pin-headers
Parts:
- added J? (x2): Conn_02x08_Odd_Even, symbol Connector_Generic:Conn_02x08_Odd_Even
Connections:
- net labels removed: IN1_N, IN1_P
- wire segments 92 -> 106
- no-connect marks 64 -> 50
Changed lines of the file:
@@
 L project_symbols:X1G0044810050_SG7050CAN_2.048_MHZ X1
 U 1 1 5B452FB5
-P 5950 4600
-F 0 "X1" H 5950 4925 50  0000 C CNN
-F 1 "X1G0044810050_SG7050CAN_2.048_MHZ" H 5950 4834 50  0000 C CNN
-F 2 "prj_lib_fp:SG0705" H 5900 4600 50  0001 C CNN
-F 3 "http://www.farnell.com/datasheets/1841779.pdf" H 5250 5050 50  0001 C CNN
-F 4 "2442953" H 4450 5150 50  0001 C CNN "Farnell Part"
-F 5 "http://se.farnell.com/epson/x1g0044810050-sg7050can-2-048-mhz/oscillator-spxo-sg7050can-2-048/dp/2442953" H 6650 5250 50  0001 C CNN "Farnell URL"
-	1    5950 4600
+P 5300 4600
+F 0 "X1" H 5300 4925 50  0000 C CNN
+F 1 "X1G0044810050_SG7050CAN_2.048_MHZ" H 5300 4834 50  0000 C CNN
+F 2 "prj_lib_fp:SG0705" H 5250 4600 50  0001 C CNN
+F 3 "http://www.farnell.com/datasheets/1841779.pdf" H 4600 5050 50  0001 C CNN
+F 4 "2442953" H 3800 5150 50  0001 C CNN "Farnell Part"
+F 5 "http://se.farnell.com/epson/x1g0044810050-sg7050can-2-048-mhz/oscillator-spxo-sg7050can-2-048/dp/2442953" H 6000 5250 50  0001 C CNN "Farnell URL"
+	1    5300 4600
 	1    0    0    -1
 $EndComp
@@
 	-800 950  -800 1150
 Wire Wire Line
-	5050 4500 5400 4500
-Wire Wire Line
-	5400 4650 5400 4500
-Connection ~ 5400 4500
-Wire Wire Line
-	6600 4650 6500 4650
+	4400 4500 4750 4500
+Wire Wire Line
+	4750 4650 4750 4500
+Connection ~ 4750 4500
+Wire Wire Line
+	5950 4650 5850 4650
 NoConn ~ 1250 1200
 NoConn ~ 1250 1300
@@
 L Device:C_Small C1
 U 1 1 5B46310B
-P 5950 4900
-F 0 "C1" V 6050 4900 50  0000 C CNN
-F 1 "0.1uF" V 5850 4900 50  0000 C CNN
-F 2 "Capacitors_SMD:C_0805_HandSoldering" H 5950 4900 50  0001 C CNN
-F 3 "~" H 5950 4900 50  0001 C CNN
-	1    5950 4900
+P 5300 4900
+F 0 "C1" V 5400 4900 50  0000 C CNN
+F 1 "0.1uF" V 5200 4900 50  0000 C CNN
+F 2 "Capacitors_SMD:C_0805_HandSoldering" H 5300 4900 50  0001 C CNN
+F 3 "~" H 5300 4900 50  0001 C CNN
+	1    5300 4900
 	0    -1   -1   0
 $EndComp
 Wire Wire Line
-	6600 4650 6600 4900
-Wire Wire Line
-	6050 4900 6600 4900
-Connection ~ 6600 4900
-Wire Wire Line
-	6600 4900 6600 5000
-Wire Wire Line
-	5850 4900 5400 4900
-Wire Wire Line
-	5400 4900 5400 4650
-Connection ~ 5400 4650
+	5950 4650 5950 4900
+Wire Wire Line
+	5400 4900 5950 4900
+Connection ~ 5950 4900
+Wire Wire Line
+	5950 4900 5950 5000
+Wire Wire Line
+	5200 4900 4750 4900
+Wire Wire Line
+	4750 4900 4750 4650
+Connection ~ 4750 4650
 $Comp
 L power:PWR_FLAG #FLG0103
@@
 	-1150 950  -1150 1150
 Wire Wire Line
-	6500 4500 8650 4500
+	5850 4500 8650 4500
 $Comp
 L project_symbols:ADS1299-4PAG U1
@@
 +3V3
 Wire Wire Line
-	10450 5200 10550 5200
-Wire Wire Line
 	10550 5200 10550 5300
 $Comp
@@
 L power:GNDD #PWR0107
 U 1 1 5B466EBF
-P 6600 5000
-F 0 "#PWR0107" H 6600 4750 50  0001 C CNN
-F 1 "GNDD" H 6604 4845 50  0000 C CNN
-F 2 "" H 6600 5000 50  0001 C CNN
-F 3 "" H 6600 5000 50  0001 C CNN
-	1    6600 5000
+P 5950 5000
+F 0 "#PWR0107" H 5950 4750 50  0001 C CNN
+F 1 "GNDD" H 5954 4845 50  0000 C CNN
+F 2 "" H 5950 5000 50  0001 C CNN
+F 3 "" H 5950 5000 50  0001 C CNN
+	1    5950 5000
 	1    0    0    -1
 $EndComp
@@
 NoConn ~ 8650 5200
 NoConn ~ 8650 4600
-NoConn ~ 8650 2400
-NoConn ~ 8650 2500
-NoConn ~ 8650 2600
-NoConn ~ 8650 2700
-NoConn ~ 8650 2800
-NoConn ~ 8650 2900
-NoConn ~ 8650 3000
-NoConn ~ 8650 3100
-NoConn ~ 8650 3400
-NoConn ~ 8650 3500
-NoConn ~ 8650 3600
-NoConn ~ 8650 3700
 NoConn ~ 8650 4000
 NoConn ~ 8650 4100
@@
 Text Label 11200 2800 2    50   ~ 0
 DVDD
-Text Label 5050 4500 0    50   ~ 0
+Text Label 4400 4500 0    50   ~ 0
 DVDD
 Wire Notes Line
-	5000 4200 6800 4200
-Wire Notes Line
-	6800 4200 6800 5250
-Wire Notes Line
-	6800 5250 5000 5250
-Wire Notes Line
-	5000 5250 5000 4200
-Text Notes 5000 4200 0    50   ~ 0
+	4350 4200 6150 4200
+Wire Notes Line
+	6150 4200 6150 5250
+Wire Notes Line
+	6150 5250 4350 5250
+Wire Notes Line
+	4350 5250 4350 4200
+Text Notes 4350 4200 0    50   ~ 0
 External Oscillator
 $Comp
@@
 Text Notes 7150 3850 2    50   ~ 0
 RESET can be trig'd via SPI cmd.\nPWDN only possible in HW.
-Text Label 7800 3900 0    50   ~ 0
-IN1_P
-Text Label 7800 3800 0    50   ~ 0
-IN1_N
-Wire Wire Line
-	7800 3800 8650 3800
-Wire Wire Line
-	8650 3900 7800 3900
-NoConn ~ 8650 3300
-NoConn ~ 8650 3200
+$Comp
+L Connector_Generic:Conn_02x08_Odd_Even J?
+U 1 1 5B4BB278
+P 8050 3500
+F 0 "J?" H 8100 4017 50  0000 C CNN
+F 1 "Conn_02x08_Odd_Even" H 8100 3926 50  0000 C CNN
+F 2 "" H 8050 3500 50  0001 C CNN
+F 3 "~" H 8050 3500 50  0001 C CNN
+	1    8050 3500
+	1    0    0    -1
+$EndComp
+$Comp
+L Connector_Generic:Conn_02x08_Odd_Even J?
+U 1 1 5B4BB482
+P 7350 2700
+F 0 "J?" H 7400 3217 50  0000 C CNN
+F 1 "Conn_02x08_Odd_Even" H 7400 3126 50  0000 C CNN
+F 2 "" H 7350 2700 50  0001 C CNN
+F 3 "~" H 7350 2700 50  0001 C CNN
+	1    7350 2700
+	1    0    0    -1
+$EndComp
+Wire Wire Line
+	10450 5200 10550 5200
+Wire Wire Line
+	8350 3200 8650 3200
+Wire Wire Line
+	8350 3300 8650 3300
+Wire Wire Line
+	8350 3400 8650 3400
+Wire Wire Line
+	8350 3500 8650 3500
+Wire Wire Line
+	8350 3600 8650 3600
+Wire Wire Line
+	8350 3700 8650 3700
+Wire Wire Line
+	8350 3800 8650 3800
+Wire Wire Line
+	8350 3900 8650 3900
+Wire Wire Line
+	7650 2400 8650 2400
+Wire Wire Line
+	7650 2500 8650 2500
+Wire Wire Line
+	7650 2600 8650 2600
+Wire Wire Line
+	7650 2700 8650 2700
+Wire Wire Line
+	7650 2800 8650 2800
+Wire Wire Line
+	7650 2900 8650 2900
+Wire Wire Line
+	7650 3000 8650 3000
+Wire Wire Line
+	7650 3100 8650 3100
 $EndSCHEMATC

Commit message: gettin paranoid about .... crashes!
Parts:
- added C?: 1.5nF, symbol Device:C
- added C?: 10uF, symbol Device:CP
- added C? (x2): 100nF, symbol Device:C
- added C?: 100uF, symbol Device:CP
- added C? (x3): 1uF, symbol Device:C
- added R?: 1M, symbol Device:R
- J2, J3: renamed from J?; footprint (none) -> Pin_Headers:Pin_Header_Straight_2x08_Pitch2.54mm
- P1: Description (none) -> Raspberry Pi 2/3 B+ 40-pin GPIO Header
Connections:
- net labels added: BIASIN, BIASINV, BIASOUT, BIASREF, GNDA, START, VCAP1, VCAP2, VCAP3, VCAP4, VDDA, VREFN, VREFP, VSSA, XTAL
- net labels removed: +3.3V
- wire segments 106 -> 152
- no-connect marks 50 -> 35
Other:
- note added: "ADC Bypassing/Filtering"
- note added: "Bias Signals\nCHECK THIS SHIT"
- note added: "MISC."
- note added: "PIN HEADERS"
- note added: "Power Nets/DRC"
- note added: "RESET/PWDN config."
- note added: "Raspberry Pi 2/3 GPIO Header"
- note added: "Tantalum?"

Commit message: created analog/digital power symbols (copy&pasted between files)
Parts:
- added C?: 1uF, symbol Device:C
Connections:
- net labels added: AVDD, AVDD1, AVDD@2, AVSS, AVSS@1, AVSS@2, ~DRDY
- net labels removed: VDDA
- wire segments 152 -> 160
- no-connect marks 35 -> 29
Other:
- note added: "<-Charge pump analog ground."
- note added: "<-Charge pump analog supply. \nConnect 1uF to AVSS@2, pin 58."
Changed lines of the file:
@@
 NoConn ~ 10450 3700
 NoConn ~ 10450 4400
-NoConn ~ 10450 4900
-NoConn ~ 10450 5000
-NoConn ~ 10450 5100
-NoConn ~ 10450 2500
-NoConn ~ 10450 2600
-NoConn ~ 10450 2700
 Wire Notes Line
 	12900 850  12900 1850
@@
 Text Label 4300 2650 2    50   ~ 0
 BIASREF
-$Comp
-L power:GNDA #PWR?
-U 1 1 5B5C9A56
-P 1750 1150
-F 0 "#PWR?" H 1750 900 50  0001 C CNN
-F 1 "GNDA" H 1755 977 50  0000 C CNN
-F 2 "" H 1750 1150 50  0001 C CNN
-F 3 "" H 1750 1150 50  0001 C CNN
-	1    1750 1150
-	-1   0    0    1
-$EndComp
 Wire Wire Line
 	1750 1150 1750 1350
@@
 	8650 4900 8650 5000
 Wire Wire Line
-	8650 4600 7800 4600
-Text Label 7800 4600 0    50   ~ 0
+	8650 4600 7500 4600
+Text Label 7500 4600 0    50   ~ 0
 START
 Text Label 8300 4000 0    50   ~ 0
@@
 Connection ~ 13100 6400
 $Comp
-L power:VSSA #PWR?
-U 1 1 5B68FA16
-P 2000 1150
-F 0 "#PWR?" H 2000 1000 50  0001 C CNN
-F 1 "VSSA" H 2017 1323 50  0000 C CNN
-F 2 "" H 2000 1150 50  0001 C CNN
-F 3 "" H 2000 1150 50  0001 C CNN
-	1    2000 1150
-	1    0    0    -1
-$EndComp
-$Comp
-L power:VDDA #PWR?
-U 1 1 5B68FB64
-P 2250 1150
-F 0 "#PWR?" H 2250 1000 50  0001 C CNN
-F 1 "VDDA" H 2267 1323 50  0000 C CNN
-F 2 "" H 2250 1150 50  0001 C CNN
-F 3 "" H 2250 1150 50  0001 C CNN
-	1    2250 1150
-	1    0    0    -1
-$EndComp
-$Comp
 L power:PWR_FLAG #FLG?
 U 1 1 5B68FB98
@@
 Text Notes 13400 6700 0    50   ~ 0
 Tantalum?
+Wire Wire Line
+	10450 5100 11200 5100
+Wire Wire Line
+	10450 5000 11200 5000
+Text Label 11200 5000 2    50   ~ 0
+AVSS@2
+Wire Wire Line
+	10450 4900 11200 4900
+Text Label 11200 4900 2    50   ~ 0
+AVSS@1
+Text Label 11550 4500 2    50   ~ 0
+~DRDY
+Wire Wire Line
+	11550 4500 10450 4500
+Wire Wire Line
+	10450 2700 11200 2700
+Text Label 11200 2700 2    50   ~ 0
+AVDD1
+Text Notes 10850 2650 0    39   ~ 0
+<-Charge pump analog supply. \nConnect 1uF to AVSS@2, pin 58.
+Text Label 10500 2600 0    50   ~ 0
+AVDD@2
+Wire Wire Line
+	10450 2600 10500 2600
+Text Notes 11250 5000 0    50   ~ 0
+<-Charge pump analog ground.
+Text Label 13850 9000 0    50   ~ 0
+AVSS@2
+Text Label 12900 9000 2    50   ~ 0
+AVDD@2
+$Comp
+L Device:C C?
+U 1 1 5B873DA5
+P 13250 9000
+F 0 "C?" V 12998 9000 50  0000 C CNN
+F 1 "1uF" V 13089 9000 50  0000 C CNN
+F 2 "" H 13288 8850 50  0001 C CNN
+F 3 "~" H 13250 9000 50  0001 C CNN
+	1    13250 9000
+	0    1    1    0
+$EndComp
+Wire Wire Line
+	12900 9000 13100 9000
+Wire Wire Line
+	13400 9000 13850 9000
+$Comp
+L project_symbols:AVDD #PWR?
+U 1 1 5B483C31
+P 2250 1150
+F 0 "#PWR?" H 2250 1000 50  0001 C CNN
+F 1 "AVDD" H 2267 1323 50  0000 C CNN
+F 2 "" H 2250 1150 50  0001 C CNN
+F 3 "" H 2250 1150 50  0001 C CNN
+	1    2250 1150
+	1    0    0    -1
+$EndComp
+$Comp
+L project_symbols:AVSS #PWR?
+U 1 1 5B483CC3
+P 2000 1150
+F 0 "#PWR?" H 2000 1000 50  0001 C CNN
+F 1 "AVSS" H 2017 1323 50  0000 C CNN
+F 2 "" H 2000 1150 50  0001 C CNN
+F 3 "" H 2000 1150 50  0001 C CNN
+	1    2000 1150
+	1    0    0    -1
+$EndComp
 $EndSCHEMATC
