File: mobilt_eeg_frontend-exjobb2018/mobilt_eeg_frontend-exjobb2018.sch (KiCad schematic (older format))
At the start: 23 parts, among them J1 Conn_02x04_Odd_Even, J2 Conn_02x08_Odd_Even, J3 Conn_02x08_Odd_Even, P1 Conn_02x20_Odd_Even, U1 ADS1299-4PAG, X1 X1G0044810050_SG7050CAN_2.048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

Commit message: that's enough for now. Next: read datasheets thoroughly
Parts:
- added C? (x8): 4.7nF, symbol Device:C_Small
- added C? (x8): 10uF, symbol Device:C
- added C? (x4): 1uF, symbol Device:C
- added C? (x4): 100nF, symbol Device:C
- added C? (x3): 10nF, symbol Device:C
- added C? (x4): 2.2uF, symbol Device:C
- added C?: 1uF, symbol Device:C_Small
- added J?: Conn_02x20_Odd_Even, symbol Connector_Generic:Conn_02x20_Odd_Even
- added J?: Conn_01x04, symbol Connector_Generic:Conn_01x04
- added R? (x8): 4.99k 1%, symbol Device:R_Small
- added SW? (x2): SW_DIP_x01, symbol Switch:SW_DIP_x01
- added U?: TPS73233DBVT, SOT95P280X145-5N, symbol project_symbols:TPS73233DBVT
- added U?: TPS73225DBVT, SOT95P280X145-5N, symbol project_symbols:TPS73225DBVT
- added U?: TPS72325DBVT, SOT95P280X145-5N, symbol project_symbols:TPS72325DBVT
- added U?: TPS60403DBVR, SOT95P280X145-5N, symbol project_symbols:TPS60403DBVR
- C1: value 0.1uF -> 100nF
Connections:
- net labels added: -5V_unreg, AGND, DGND
- wire segments 160 -> 253
- no-connect marks 29 -> 28
Other:
- note added: "Analog Power Supplies (+/-2V5, -5V)"
- note added: "Digital Power Supply (+3V3)"
- note added: "Electrode Headers"
- note added: "RasPi I2C Header"
- note added: "RasPi Tactile Buttons"

Commit message: done some stuff... it would be a shame if anything happened to it....
Parts:
- removed C? (x8): 4.7nF, symbol Device:C_Small
- removed R? (x8): 4.99k 1%, symbol Device:R_Small
- added C?: 1uF, Capacitors_SMD:C_0805_HandSoldering, symbol Device:C_Small
- added C? (x10): 4.7nF, symbol Device:C_Small
- added D?: LED, symbol Device:LED
- added J?: Conn_01x08, symbol Connector_Generic:Conn_01x08
- added J?: Conn_01x10, symbol Connector_Generic:Conn_01x10
- added J?: Conn_01x01, symbol Connector_Generic:Conn_01x01
- added J?: Conn_01x02, symbol Connector_Generic:Conn_01x02
- added R?: 1k, symbol Device:R
- added R? (x10): 4.99k 1%, symbol Device:R_Small
- added R?: 10k, symbol Device:R
- added R? (x2): 3.9k, symbol Device:R
- added U?: CAT24C256, symbol Memory_EEPROM:CAT24C256
Connections:
- net labels added: AVDD@1, IN1N, IN1P, IN2N, IN2P, IN3N, IN3P, IN4N, IN4P, IN5N, IN5P, IN6N, IN6P, IN7N, IN7P, IN8N, IN8P, SRB1, SRB2
- wire segments 253 -> 307
- no-connect marks 28 -> 26
Other:
- note added: "1uF not mentioned in datasheet"
- note added: "Power Rails Header"
- note added: "RasPi HAT-compliant EEPROM"
- note added: "RasPi Status LED"
- note added: "Test Point -5V"
- note added: "WE Jumper"
